File: tessel-v2-coprocessor.sch (KiCad schematic (older format))
At the start: 22 parts

Commit message: annotated
Parts:
- gave numbers to parts that had none: 22
Changed lines of the file:
@@
 PORT_B_G3
 $Comp
-L C C?
+L C C804
 U 1 1 548F96CA
 P 6000 7750
-F 0 "C?" H 6000 7850 40  0000 L CNN
+F 0 "C804" H 6000 7850 40  0000 L CNN
 F 1 "10pF" H 6006 7665 40  0000 L CNN
 F 2 "" H 6038 7600 30  0000 C CNN
@@
 $EndComp
 $Comp
-L C C?
+L C C802
 U 1 1 548F96F8
 P 4800 7750
-F 0 "C?" H 4800 7850 40  0000 L CNN
+F 0 "C802" H 4800 7850 40  0000 L CNN
 F 1 "10pF" H 4806 7665 40  0000 L CNN
 F 2 "" H 4838 7600 30  0000 C CNN
@@
 $EndComp
 $Comp
-L GND #PWR?
+L GND #PWR802
 U 1 1 548F9730
 P 4800 8100
-F 0 "#PWR?" H 4800 8100 30  0001 C CNN
+F 0 "#PWR802" H 4800 8100 30  0001 C CNN
 F 1 "GND" H 4800 8030 30  0001 C CNN
 F 2 "" H 4800 8100 60  0000 C CNN
@@
 $EndComp
 $Comp
-L GND #PWR?
+L GND #PWR804
 U 1 1 548F973F
 P 6000 8100
-F 0 "#PWR?" H 6000 8100 30  0001 C CNN
+F 0 "#PWR804" H 6000 8100 30  0001 C CNN
 F 1 "GND" H 6000 8030 30  0001 C CNN
 F 2 "" H 6000 8100 60  0000 C CNN
@@
 12.5pF\nNOMINAL\nSHUNT
 $Comp
-L C C?
+L C C808
 U 1 1 548F9D44
 P 7500 3650
-F 0 "C?" H 7500 3750 40  0000 L CNN
+F 0 "C808" H 7500 3750 40  0000 L CNN
 F 1 "10uF" H 7506 3565 40  0000 L CNN
 F 2 "" H 7538 3500 30  0000 C CNN
@@
 $EndComp
 $Comp
-L C C?
+L C C810
 U 1 1 548F9D6C
 P 9350 3600
-F 0 "C?" H 9350 3700 40  0000 L CNN
+F 0 "C810" H 9350 3700 40  0000 L CNN
 F 1 "100nF" H 9356 3515 40  0000 L CNN
 F 2 "" H 9388 3450 30  0000 C CNN
@@
 $EndComp
 $Comp
-L INDUCTOR L?
+L INDUCTOR L801
 U 1 1 548FA5A7
 P 8600 2850
-F 0 "L?" V 8550 2850 40  0000 C CNN
+F 0 "L801" V 8550 2850 40  0000 C CNN
 F 1 "10uH" V 8700 2850 40  0000 C CNN
 F 2 "" H 8600 2850 60  0000 C CNN
@@
 $EndComp
 $Comp
-L C C?
+L C C805
 U 1 1 548FA741
 P 6300 3650
-F 0 "C?" H 6300 3750 40  0000 L CNN
+F 0 "C805" H 6300 3750 40  0000 L CNN
 F 1 "100nF" H 6306 3565 40  0000 L CNN
 F 2 "" H 6338 3500 30  0000 C CNN
@@
 $EndComp
 $Comp
-L C C?
+L C C807
 U 1 1 548FA7B7
 P 7100 3650
-F 0 "C?" H 7100 3750 40  0000 L CNN
+F 0 "C807" H 7100 3750 40  0000 L CNN
 F 1 "100nF" H 7106 3565 40  0000 L CNN
 F 2 "" H 7138 3500 30  0000 C CNN
@@
 $EndComp
 $Comp
-L C C?
+L C C806
 U 1 1 548FA7E4
 P 6700 3650
-F 0 "C?" H 6700 3750 40  0000 L CNN
+F 0 "C806" H 6700 3750 40  0000 L CNN
 F 1 "100nF" H 6706 3565 40  0000 L CNN
 F 2 "" H 6738 3500 30  0000 C CNN
@@
 $EndComp
 $Comp
-L C C?
+L C C803
 U 1 1 548FAA8B
 P 5900 3650
-F 0 "C?" H 5900 3750 40  0000 L CNN
+F 0 "C803" H 5900 3750 40  0000 L CNN
 F 1 "100nF" H 5906 3565 40  0000 L CNN
 F 2 "" H 5938 3500 30  0000 C CNN
@@
 $EndComp
 $Comp
-L C C?
+L C C809
 U 1 1 548FAB15
 P 8950 3600
-F 0 "C?" H 8950 3700 40  0000 L CNN
+F 0 "C809" H 8950 3700 40  0000 L CNN
 F 1 "10uF" H 8956 3515 40  0000 L CNN
 F 2 "" H 8988 3450 30  0000 C CNN
@@
 $EndComp
 $Comp
-L SAMD21G14A-MU U?
+L SAMD21G14A-MU U801
 U 1 1 548FAB63
 P 8300 6000
-F 0 "U?" H 7150 7650 40  0000 C CNN
+F 0 "U801" H 7150 7650 40  0000 C CNN
 F 1 "SAMD21G14A-MU" H 8300 6000 40  0000 C CNN
 F 2 "QFN48" H 8300 5900 32  0000 C CIN
@@
 VDDIN
 $Comp
-L GND #PWR?
+L GND #PWR811
 U 1 1 548FA205
 P 9350 4000
-F 0 "#PWR?" H 9350 4000 30  0001 C CNN
+F 0 "#PWR811" H 9350 4000 30  0001 C CNN
 F 1 "GND" H 9350 3930 30  0001 C CNN
 F 2 "" H 9350 4000 60  0000 C CNN
@@
 $EndComp
 $Comp
-L GND #PWR?
+L GND #PWR810
 U 1 1 548FBD70
 P 8950 4000
-F 0 "#PWR?" H 8950 4000 30  0001 C CNN
+F 0 "#PWR810" H 8950 4000 30  0001 C CNN
 F 1 "GND" H 8950 3930 30  0001 C CNN
 F 2 "" H 8950 4000 60  0000 C CNN
@@
 $EndComp
 $Comp
-L GND #PWR?
+L GND #PWR808
 U 1 1 548FBD83
 P 7500 4050
-F 0 "#PWR?" H 7500 4050 30  0001 C CNN
+F 0 "#PWR808" H 7500 4050 30  0001 C CNN
 F 1 "GND" H 7500 3980 30  0001 C CNN
 F 2 "" H 7500 4050 60  0000 C CNN
@@
 $EndComp
 $Comp
-L GND #PWR?
+L GND #PWR807
 U 1 1 548FBD8A
 P 7100 4050
-F 0 "#PWR?" H 7100 4050 30  0001 C CNN
+F 0 "#PWR807" H 7100 4050 30  0001 C CNN
 F 1 "GND" H 7100 3980 30  0001 C CNN
 F 2 "" H 7100 4050 60  0000 C CNN
@@
 $EndComp
 $Comp
-L GND #PWR?
+L GND #PWR806
 U 1 1 548FBD9D
 P 6700 4050
-F 0 "#PWR?" H 6700 4050 30  0001 C CNN
+F 0 "#PWR806" H 6700 4050 30  0001 C CNN
 F 1 "GND" H 6700 3980 30  0001 C CNN
 F 2 "" H 6700 4050 60  0000 C CNN
@@
 $EndComp
 $Comp
-L GND #PWR?
+L GND #PWR805
 U 1 1 548FBDA4
 P 6300 4050
-F 0 "#PWR?" H 6300 4050 30  0001 C CNN
+F 0 "#PWR805" H 6300 4050 30  0001 C CNN
 F 1 "GND" H 6300 3980 30  0001 C CNN
 F 2 "" H 6300 4050 60  0000 C CNN
@@
 $EndComp
 $Comp
-L GND #PWR?
+L GND #PWR803
 U 1 1 548FBDB7
 P 5900 4050
-F 0 "#PWR?" H 5900 4050 30  0001 C CNN
+F 0 "#PWR803" H 5900 4050 30  0001 C CNN
 F 1 "GND" H 5900 3980 30  0001 C CNN
 F 2 "" H 5900 4050 60  0000 C CNN
@@
 Connection ~ 7500 3250
 $Comp
-L GND #PWR?
+L GND #PWR809
 U 1 1 548FD791
 P 8000 8100
-F 0 "#PWR?" H 8000 8100 30  0001 C CNN
+F 0 "#PWR809" H 8000 8100 30  0001 C CNN
 F 1 "GND" H 8000 8030 30  0001 C CNN
 F 2 "" H 8000 8100 60  0000 C CNN
@@
 VDDANA
 $Comp
-L CRYSTAL X?
+L CRYSTAL X801
 U 1 1 54900866
 P 5400 7400
-F 0 "X?" H 5400 7550 60  0000 C CNN
+F 0 "X801" H 5400 7550 60  0000 C CNN
 F 1 "SC32S-12.5PF20PPM" H 5400 7250 60  0000 C CNN
 F 2 "" H 5400 7400 60  0000 C CNN
@@
 MT_PWR_EN
 $Comp
-L R R?
+L R R804
 U 1 1 54912B30
 P 12300 6200
-F 0 "R?" V 12380 6200 40  0000 C CNN
+F 0 "R804" V 12380 6200 40  0000 C CNN
 F 1 "22R" V 12307 6201 40  0000 C CNN
 F 2 "" V 12230 6200 30  0000 C CNN
@@
 $EndComp
 $Comp
-L R R?
+L R R805
 U 1 1 54912C7C
 P 12300 6400
-F 0 "R?" V 12380 6400 40  0000 C CNN
+F 0 "R805" V 12380 6400 40  0000 C CNN
 F 1 "22R" V 12307 6401 40  0000 C CNN
 F 2 "" V 12230 6400 30  0000 C CNN
@@
 $EndComp
 $Comp
-L R R?
+L R R802
 U 1 1 54912D2C
 P 12300 5800
-F 0 "R?" V 12380 5800 40  0000 C CNN
+F 0 "R802" V 12380 5800 40  0000 C CNN
 F 1 "22R" V 12307 5801 40  0000 C CNN
 F 2 "" V 12230 5800 30  0000 C CNN
@@
 $EndComp
 $Comp
-L R R?
+L R R803
 U 1 1 54912D32
 P 12300 6000
-F 0 "R?" V 12380 6000 40  0000 C CNN
+F 0 "R803" V 12380 6000 40  0000 C CNN
 F 1 "22R" V 12307 6001 40  0000 C CNN
 F 2 "" V 12230 6000 30  0000 C CNN
@@
 	9700 6900 11800 6900
 $Comp
-L R R?
+L R R807
 U 1 1 54913EBE
 P 12300 6800
-F 0 "R?" V 12380 6800 40  0000 C CNN
+F 0 "R807" V 12380 6800 40  0000 C CNN
 F 1 "22R" V 12307 6801 40  0000 C CNN
 F 2 "" V 12230 6800 30  0000 C CNN
@@
 $EndComp
 $Comp
-L R R?
+L R R806
 U 1 1 54913EC4
 P 12300 6600
-F 0 "R?" V 12380 6600 40  0000 C CNN
+F 0 "R806" V 12380 6600 40  0000 C CNN
 F 1 "22R" V 12307 6601 40  0000 C CNN
 F 2 "" V 12230 6600 30  0000 C CNN
@@
 $EndComp
 $Comp
-L R R?
+L R R809
 U 1 1 54913ECA
 P 12300 7200
-F 0 "R?" V 12380 7200 40  0000 C CNN
+F 0 "R809" V 12380 7200 40  0000 C CNN
 F 1 "22R" V 12307 7201 40  0000 C CNN
 F 2 "" V 12230 7200 30  0000 C CNN
@@
 $EndComp
 $Comp
-L R R?
+L R R808
 U 1 1 54913ED0
 P 12300 7000
-F 0 "R?" V 12380 7000 40  0000 C CNN
+F 0 "R808" V 12380 7000 40  0000 C CNN
 F 1 "22R" V 12307 7001 40  0000 C CNN
 F 2 "" V 12230 7000 30  0000 C CNN
@@
 	3150 4600 4100 4600
 $Comp
-L C C?
+L C C801
 U 1 1 54978225
 P 4100 4900
-F 0 "C?" H 4100 5000 40  0000 L CNN
+F 0 "C801" H 4100 5000 40  0000 L CNN
 F 1 "100nF" H 4106 4815 40  0000 L CNN
 F 2 "" H 4138 4750 30  0000 C CNN
@@
 	4100 5100 4100 5200
 $Comp
-L R R?
+L R R801
 U 1 1 5497863A
 P 4100 4250
-F 0 "R?" V 4180 4250 40  0000 C CNN
+F 0 "R801" V 4180 4250 40  0000 C CNN
 F 1 "22R" V 4107 4251 40  0000 C CNN
 F 2 "" V 4030 4250 30  0000 C CNN
@@
 3.3V_CP
 $Comp
-L GND #PWR?
+L GND #PWR801
 U 1 1 54978E0E
 P 4100 5200
-F 0 "#PWR?" H 4100 5200 30  0001 C CNN
+F 0 "#PWR801" H 4100 5200 30  0001 C CNN
 F 1 "GND" H 4100 5130 30  0001 C CNN
 F 2 "" H 4100 5200 60  0000 C CNN
