File: tessel-v2-mediatek-rf.sch (KiCad schematic (older format))
At the start: 45 parts, among them J501 CONN_01X01, J502 CONN_01X01, J503 CONN_01X03, U201 MT7620N

Commit message: starting cvpcb
Parts:
- AE501, AE502: footprint (none) -> tm-kicad-lib:ANTENNA-SMT-2.45GHz
- AE503, AE504: footprint (none) -> tm-kicad-lib:1909763-1
