File: tessel-v2-mediatek-rf.sch (KiCad schematic (older format))
At the start: 43 parts, among them J501 CONN_01X01, J502 CONN_01X01, T501 2450BL15B100, T502 2450BL15B100, U201 MT7620N

Commit message: datasheets, refdes, netlists, and component mappings
Parts:
- R501: value 24kR, 1% -> 24kR 1%
- R504: value 4.7kR, 1% -> 4.7kR 1%
- R505: value 4.7kR, DNP -> 4.7kR DNP
Changed lines of the file:
@@
 P 2050 5500
 F 0 "R501" V 2130 5500 40  0000 C CNN
-F 1 "24kR, 1%" V 2057 5501 40  0000 C CNN
+F 1 "24kR 1%" V 2057 5501 40  0000 C CNN
 F 2 "tm-kicad-lib:SMD-0402" V 1980 5500 30  0001 C CNN
 F 3 "" H 2050 5500 30  0000 C CNN
@@
 P 4900 5350
 F 0 "R505" V 4980 5350 40  0000 C CNN
-F 1 "4.7kR, DNP" V 4907 5351 40  0000 C CNN
+F 1 "4.7kR DNP" V 4907 5351 40  0000 C CNN
 F 2 "tm-kicad-lib:SMD-0402" V 4830 5350 30  0001 C CNN
 F 3 "" H 4900 5350 30  0000 C CNN
@@
 P 4750 5350
 F 0 "R504" V 4830 5350 40  0000 C CNN
-F 1 "4.7kR, 1%" V 4757 5351 40  0000 C CNN
+F 1 "4.7kR 1%" V 4757 5351 40  0000 C CNN
 F 2 "tm-kicad-lib:SMD-0402" V 4680 5350 30  0001 C CNN
 F 3 "" H 4750 5350 30  0000 C CNN

Commit message: 1%, DNP, etc
Parts:
- T501, T502: footprint (none) -> !Parts:EIA-0805
Changed lines of the file:
@@
 F 0 "T501" H 9250 4300 60  0000 C CNN
 F 1 "2450BL15B100" H 9600 4000 60  0000 C CNN
-F 2 "" H 9600 3950 60  0001 C CNN
+F 2 "!Parts:EIA-0805" H 9600 3950 60  0001 C CNN
 F 3 "" H 9600 3950 60  0000 C CNN
 	1    9600 3950
@@
 F 0 "T502" H 9250 8150 60  0000 C CNN
 F 1 "2450BL15B100" H 9600 7850 60  0000 C CNN
-F 2 "" H 9600 7800 60  0001 C CNN
+F 2 "!Parts:EIA-0805" H 9600 7800 60  0001 C CNN
 F 3 "" H 9600 7800 60  0000 C CNN
 	1    9600 7800
