File: tessel-v2.sch (KiCad schematic (older format))
At the start: 0 parts

Commit message: added mount holes, 3" guide lines... it will be a miracle if it fits
Parts:
- added H101, H102, H103, H104: HOLE, Mounting_Holes:MountingHole_2-5mm, symbol HOLE
Changed lines of the file:
@@
 Wire Wire Line
 	9000 5250 10800 5250
+$Comp
+L HOLE H101
+U 1 1 54C07487
+P 2900 9400
+F 0 "H101" H 2900 9550 60  0000 C CNN
+F 1 "HOLE" H 2900 9250 60  0000 C CNN
+F 2 "Mounting_Holes:MountingHole_2-5mm" H 2900 9400 60  0001 C CNN
+F 3 "" H 2900 9400 60  0000 C CNN
+	1    2900 9400
+	1    0    0    -1
+$EndComp
+$Comp
+L HOLE H102
+U 1 1 54C07804
+P 3200 9400
+F 0 "H102" H 3200 9550 60  0000 C CNN
+F 1 "HOLE" H 3200 9250 60  0000 C CNN
+F 2 "Mounting_Holes:MountingHole_2-5mm" H 3200 9400 60  0001 C CNN
+F 3 "" H 3200 9400 60  0000 C CNN
+	1    3200 9400
+	1    0    0    -1
+$EndComp
+$Comp
+L HOLE H103
+U 1 1 54C07827
+P 3500 9400
+F 0 "H103" H 3500 9550 60  0000 C CNN
+F 1 "HOLE" H 3500 9250 60  0000 C CNN
+F 2 "Mounting_Holes:MountingHole_2-5mm" H 3500 9400 60  0001 C CNN
+F 3 "" H 3500 9400 60  0000 C CNN
+	1    3500 9400
+	1    0    0    -1
+$EndComp
+$Comp
+L HOLE H104
+U 1 1 54C07848
+P 3800 9400
+F 0 "H104" H 3800 9550 60  0000 C CNN
+F 1 "HOLE" H 3800 9250 60  0000 C CNN
+F 2 "Mounting_Holes:MountingHole_2-5mm" H 3800 9400 60  0001 C CNN
+F 3 "" H 3800 9400 60  0000 C CNN
+	1    3800 9400
+	1    0    0    -1
+$EndComp
 $EndSCHEMATC

Commit message: post-schematic review. changes in.
Changed lines of the file:
@@
 F7 "MT_MOSI" I R 9000 5600 60
 F8 "MT_MISO" I R 9000 5700 60
-F9 "MT_WP" I R 9000 8600 60
 F10 "MT_SCL" I R 9000 5950 60
 F11 "MT_SDA" I R 9000 6050 60
@@
 $EndSheet
 Wire Wire Line
-	10550 7000 10550 9750
+	10550 6950 10550 9750
 Wire Wire Line
-	10550 7000 13050 7000
-Wire Wire Line
-	13050 7000 13050 6950
-Wire Wire Line
-	13050 6950 13150 6950
+	10550 6950 13150 6950
 Wire Wire Line
 	10600 7050 13150 7050
@@
 	10600 9100 9000 9100
 Wire Wire Line
-	9000 8600 9300 8600
-Wire Wire Line
-	9300 8600 9300 8450
-Connection ~ 9300 8450
-Wire Wire Line
 	6650 4650 6650 9750

Commit message: logo? logo.
Parts:
- added SILK?: logo, symbol logo
Changed lines of the file:
@@
 LIBS:valves
 LIBS:tm-kicad-lib
-LIBS:nordicsemi
 LIBS:tessel-v2-cache
 EELAYER 25 0
@@
 	1    0    0    -1
 $EndComp
+$Comp
+L logo SILK?
+U 1 1 54DD821E
+P 4200 9400
+F 0 "SILK?" H 4200 9450 60  0000 C CNN
+F 1 "logo" H 4200 9350 60  0000 C CNN
+F 2 "" H 4200 9400 60  0000 C CNN
+F 3 "" H 4200 9400 60  0000 C CNN
+	1    4200 9400
+	1    0    0    -1
+$EndComp

Commit message: done with renders for the day
Parts:
- removed SILK?: logo, symbol logo
- added SILK101: logo, !Parts:TESSEL-HEXAGON-LOGO, symbol logo
Changed lines of the file:
@@
 $EndComp
 $Comp
-L logo SILK?
-U 1 1 54DD821E
+L logo SILK101
+U 1 1 54DD9FA3
 P 4200 9400
-F 0 "SILK?" H 4200 9450 60  0000 C CNN
+F 0 "SILK101" H 4200 9450 60  0000 C CNN
 F 1 "logo" H 4200 9350 60  0000 C CNN
-F 2 "" H 4200 9400 60  0000 C CNN
+F 2 "!Parts:TESSEL-HEXAGON-LOGO" H 4200 9400 60  0001 C CNN
 F 3 "" H 4200 9400 60  0000 C CNN
 	1    4200 9400

Commit message: working towards pin muxing for v2v3 and general schematic cleanup
Changed lines of the file:
@@
 	10900 3750 13150 3750
 Wire Wire Line
-	9000 5500 10700 5500
+	9000 5500 9450 5500
+Wire Wire Line
+	9450 5500 10700 5500
 Wire Wire Line
 	10700 5500 10700 3050
@@
 	10700 3050 13150 3050
 Wire Wire Line
-	9000 5600 10600 5600
+	9000 5600 9550 5600
+Wire Wire Line
+	9550 5600 10600 5600
 Wire Wire Line
 	10600 5600 10600 2850
@@
 	10600 2850 13150 2850
 Wire Wire Line
-	9000 5700 10500 5700
+	9000 5700 9650 5700
+Wire Wire Line
+	9650 5700 10500 5700
 Wire Wire Line
 	10500 5700 10500 2950
@@
 	10600 9100 9000 9100
 Wire Wire Line
-	6650 4650 6650 9750
+	6650 4650 6650 5500
+Wire Wire Line
+	6650 5500 6650 9750
 Wire Wire Line
 	6650 9750 10550 9750
