File: tessel-v2-io.sch (KiCad schematic (older format))
At the start: 34 parts, among them J803 HR911105A, J806 CONN_01X02, J817 CONN_01X01, U201 MT7620N

Commit message: reset annotation
Parts:
- gave numbers to parts that had none: 5
- renumbered C814 to C701, C813 to C702, C822 to C703, D807 to D703, D802 to D704, J817 to J701, J803 to J702, J806 to J704, R811 to R701, R812 to R702, R813 to R703, R814 to R704, R817 to R705, R818 to R706, R815 to R707, R816 to R708, R825 to R709, R826 to R710, R833 to R711, R819 to R712, R823 to R713, R822 to R714, R827 to R716, R802 to R718, R806 to R719, R809 to R720, R829 to R721, R810 to R722

Commit message: annotation did not take?
Connections:
- wire segments 168 -> 149
Changed lines of the file:
@@
 Connection ~ 4700 8400
 Wire Wire Line
-	4700 8200 4700 8300
-Wire Wire Line
-	4700 8300 4700 8400
-Wire Wire Line
-	4700 8400 4700 8500
+	4700 8200 4700 8500
 Connection ~ 4700 8300
 Wire Wire Line
@@
 	5100 9000 5100 9100
 Wire Wire Line
-	4700 8900 4700 9100
-Wire Wire Line
-	4700 9100 4700 9200
+	4700 8900 4700 9200
 Connection ~ 13200 3800
 Wire Wire Line
@@
 Connection ~ 2300 9800
 Wire Wire Line
-	2300 9700 2300 9800
-Wire Wire Line
-	2300 9800 2300 9900
+	2300 9700 2300 9900
 Wire Wire Line
 	1900 9700 1900 9800
@@
 	2300 8200 2300 8300
 Wire Wire Line
-	1900 8100 1900 8200
-Wire Wire Line
-	1900 8200 1900 8300
+	1900 8100 1900 8300
 Connection ~ 1900 9100
 Wire Wire Line
-	1900 8800 1900 9100
-Wire Wire Line
-	1900 9100 1900 9200
+	1900 8800 1900 9200
 Wire Wire Line
 	2400 9100 1900 9100
 Connection ~ 2300 8900
 Wire Wire Line
-	2300 8800 2300 8900
-Wire Wire Line
-	2300 8900 2300 9200
+	2300 8800 2300 9200
 Wire Wire Line
 	2400 8900 2300 8900
@@
 	5300 7200 5200 7200
 Wire Wire Line
-	5300 7000 5300 7200
-Wire Wire Line
-	5300 7200 5300 7500
+	5300 7000 5300 7500
 Wire Wire Line
 	5300 7500 5200 7500
@@
 	2900 8900 3000 8900
 Wire Wire Line
-	1900 4000 2500 4000
+	1900 4000 3600 4000
 Wire Wire Line
-	2500 4000 3600 4000
+	1900 6000 3300 6000
 Wire Wire Line
-	1900 6000 2500 6000
+	13100 3500 13600 3500
 Wire Wire Line
-	2500 6000 3300 6000
-Wire Wire Line
-	13100 3500 13200 3500
-Wire Wire Line
-	13200 3500 13600 3500
-Wire Wire Line
-	13100 3600 13300 3600
-Wire Wire Line
-	13300 3600 13700 3600
+	13100 3600 13700 3600
 Wire Wire Line
 	10850 3200 11600 3200
@@
 	10600 3700 11600 3700
 Wire Wire Line
-	13200 2600 13200 2700
-Wire Wire Line
-	13200 2700 13200 3500
+	13200 2600 13200 3500
 Connection ~ 13200 3500
 Wire Wire Line
@@
 	11500 3800 11500 4000
 Wire Wire Line
-	9100 3800 11500 3800
-Wire Wire Line
-	11500 3800 11600 3800
+	9100 3800 11600 3800
 Wire Wire Line
 	11500 4500 11500 4600
 Wire Wire Line
-	1900 7600 2500 7600
+	1900 7600 3800 7600
 Wire Wire Line
-	2500 7600 3800 7600
-Wire Wire Line
-	1900 5600 2500 5600
-Wire Wire Line
-	2500 5600 3500 5600
+	1900 5600 3500 5600
 Wire Wire Line
 	5700 1800 5100 1800
@@
 	5700 2100 5100 2100
 Wire Wire Line
-	13100 3800 13200 3800
-Wire Wire Line
-	13200 3800 14700 3800
+	13100 3800 14700 3800
 Wire Wire Line
 	9700 6700 9700 6800
@@
 	6800 7300 7000 7300
 Wire Wire Line
-	2500 4600 2500 4700
-Wire Wire Line
-	2500 4700 2500 5000
+	2500 4600 2500 5000
 Wire Wire Line
 	2500 5500 2500 5600
@@
 Connection ~ 2500 6000
 Wire Wire Line
-	2500 6600 2500 6700
-Wire Wire Line
-	2500 6700 2500 7000
+	2500 6600 2500 7000
 Wire Wire Line
 	2900 6800 2900 6700

Commit message: post-quick review from refactor
Parts:
- renumbered R712 to R711, R711 to R712
Other:
- note added: "DIFF PAIR"
- moved on the sheet: C703, R712, R713, R714

Commit message: value optimization for the sake of bom complexity
Parts:
- J703: footprint (none) -> !Parts:CONN_01x08_0.05in
Changed lines of the file:
@@
 F 0 "J703" H 8400 3700 50  0000 C CNN
 F 1 "CONN_01X08" V 8500 3250 50  0000 C CNN
-F 2 "" H 8400 3250 60  0000 C CNN
+F 2 "!Parts:CONN_01x08_0.05in" H 8400 3250 60  0001 C CNN
 F 3 "" H 8400 3250 60  0000 C CNN
 	1    8400 3250

Commit message: back-propogated componet information, placed lots of things
Parts:
- J701: footprint !Parts:Testpoint -> tm-kicad-lib:Testpoint
- J703: footprint !Parts:CONN_01x08_0.05in -> tm-kicad-lib:CONN_01x08_0.05in
Changed lines of the file:
@@
 $EndComp
 $Comp
-L GND #PWR705
+L GND #PWR0160
 U 1 1 54903FAB
 P 4700 8300
-F 0 "#PWR705" H 4700 8050 60  0001 C CNN
+F 0 "#PWR0160" H 4700 8050 60  0001 C CNN
 F 1 "GND" H 4700 8150 60  0000 C CNN
 F 2 "" H 4700 8300 60  0000 C CNN
@@
 ETH_LED_GREEN
 $Comp
-L GND #PWR707
+L GND #PWR0161
 U 1 1 54945F8D
 P 5300 3350
-F 0 "#PWR707" H 5300 3100 60  0001 C CNN
+F 0 "#PWR0161" H 5300 3100 60  0001 C CNN
 F 1 "GND" H 5300 3200 60  0000 C CNN
 F 2 "" H 5300 3350 60  0000 C CNN
@@
 $EndComp
 $Comp
-L +3.3V #PWR701
+L +3.3V #PWR0162
 U 1 1 5495E2CB
 P 1900 8100
-F 0 "#PWR701" H 1900 8060 30  0001 C CNN
+F 0 "#PWR0162" H 1900 8060 30  0001 C CNN
 F 1 "+3.3V" H 1900 8210 30  0000 C CNN
 F 2 "" H 1900 8100 60  0000 C CNN
@@
 $EndComp
 $Comp
-L +3.3V #PWR713
+L +3.3V #PWR0163
 U 1 1 54925667
 P 12500 2400
-F 0 "#PWR713" H 12500 2360 30  0001 C CNN
+F 0 "#PWR0163" H 12500 2360 30  0001 C CNN
 F 1 "+3.3V" H 12500 2510 30  0000 C CNN
 F 2 "" H 12500 2400 60  0000 C CNN
@@
 $EndComp
 $Comp
-L GND #PWR712
+L GND #PWR0164
 U 1 1 54928DC4
 P 11500 4600
-F 0 "#PWR712" H 11500 4350 60  0001 C CNN
+F 0 "#PWR0164" H 11500 4350 60  0001 C CNN
 F 1 "GND" H 11500 4450 60  0000 C CNN
 F 2 "" H 11500 4600 60  0000 C CNN
@@
 F 0 "J701" H 1600 2800 50  0000 C CNN
 F 1 "CONN_01X01" V 1700 2700 50  0000 C CNN
-F 2 "!Parts:Testpoint" H 1600 2700 60  0001 C CNN
+F 2 "tm-kicad-lib:Testpoint" H 1600 2700 60  0001 C CNN
 F 3 "" H 1600 2700 60  0000 C CNN
 	1    1600 2700
@@
 $EndComp
 $Comp
-L +3.3V #PWR708
+L +3.3V #PWR0165
 U 1 1 54C65D35
 P 5700 7000
-F 0 "#PWR708" H 5700 6960 30  0001 C CNN
+F 0 "#PWR0165" H 5700 6960 30  0001 C CNN
 F 1 "+3.3V" H 5700 7110 30  0000 C CNN
 F 2 "" H 5700 7000 60  0000 C CNN
@@
 $EndComp
 $Comp
-L GND #PWR706
+L GND #PWR0166
 U 1 1 54CABBD2
 P 5100 9200
-F 0 "#PWR706" H 5100 8950 60  0001 C CNN
+F 0 "#PWR0166" H 5100 8950 60  0001 C CNN
 F 1 "GND" H 5100 9050 60  0000 C CNN
 F 2 "" H 5100 9200 60  0000 C CNN
@@
 $EndComp
 $Comp
-L GND #PWR702
+L GND #PWR0167
 U 1 1 54CAC344
 P 2300 9900
-F 0 "#PWR702" H 2300 9650 60  0001 C CNN
+F 0 "#PWR0167" H 2300 9650 60  0001 C CNN
 F 1 "GND" H 2300 9750 60  0000 C CNN
 F 2 "" H 2300 9900 60  0000 C CNN
@@
 CP_BRIDGE_SAM_RX
 $Comp
-L GND #PWR714
+L GND #PWR0168
 U 1 1 54E8E7F1
 P 12800 7900
-F 0 "#PWR714" H 12800 7650 60  0001 C CNN
+F 0 "#PWR0168" H 12800 7650 60  0001 C CNN
 F 1 "GND" H 12800 7750 60  0000 C CNN
 F 2 "" H 12800 7900 60  0000 C CNN
@@
 $EndComp
 $Comp
-L GND #PWR715
+L GND #PWR0169
 U 1 1 54E9085B
 P 13200 4600
-F 0 "#PWR715" H 13200 4350 60  0001 C CNN
+F 0 "#PWR0169" H 13200 4350 60  0001 C CNN
 F 1 "GND" H 13200 4450 60  0000 C CNN
 F 2 "" H 13200 4600 60  0000 C CNN
@@
 $EndComp
 $Comp
-L GND #PWR711
+L GND #PWR0170
 U 1 1 54EA71A9
 P 11300 7900
-F 0 "#PWR711" H 11300 7650 60  0001 C CNN
+F 0 "#PWR0170" H 11300 7650 60  0001 C CNN
 F 1 "GND" H 11300 7750 60  0000 C CNN
 F 2 "" H 11300 7900 60  0000 C CNN
@@
 $EndComp
 $Comp
-L +3.3V #PWR710
+L +3.3V #PWR0171
 U 1 1 54EC1D35
 P 9700 6700
-F 0 "#PWR710" H 9700 6660 30  0001 C CNN
+F 0 "#PWR0171" H 9700 6660 30  0001 C CNN
 F 1 "+3.3V" H 9700 6810 30  0000 C CNN
 F 2 "" H 9700 6700 60  0000 C CNN
@@
 ~WLAN~_LED
 $Comp
-L GND #PWR716
+L GND #PWR0172
 U 1 1 54ED32A7
 P 14400 7900
-F 0 "#PWR716" H 14400 7650 60  0001 C CNN
+F 0 "#PWR0172" H 14400 7650 60  0001 C CNN
 F 1 "GND" H 14400 7750 60  0000 C CNN
 F 2 "" H 14400 7900 60  0000 C CNN
@@
 RN_P1
 $Comp
-L GND #PWR703
+L GND #PWR0173
 U 1 1 54E7D87F
 P 2900 5300
-F 0 "#PWR703" H 2900 5050 60  0001 C CNN
+F 0 "#PWR0173" H 2900 5050 60  0001 C CNN
 F 1 "GND" H 2900 5150 60  0000 C CNN
 F 2 "" H 2900 5300 60  0000 C CNN
@@
 $EndComp
 $Comp
-L GND #PWR704
+L GND #PWR0174
 U 1 1 54E7E15B
 P 2900 7300
-F 0 "#PWR704" H 2900 7050 60  0001 C CNN
+F 0 "#PWR0174" H 2900 7050 60  0001 C CNN
 F 1 "GND" H 2900 7150 60  0000 C CNN
 F 2 "" H 2900 7300 60  0000 C CNN
@@
 F 0 "J703" H 8400 3700 50  0000 C CNN
 F 1 "CONN_01X08" V 8500 3250 50  0000 C CNN
-F 2 "!Parts:CONN_01x08_0.05in" H 8400 3250 60  0001 C CNN
+F 2 "tm-kicad-lib:CONN_01x08_0.05in" H 8400 3250 60  0001 C CNN
 F 3 "" H 8400 3250 60  0000 C CNN
 	1    8400 3250
@@
 $EndComp
 $Comp
-L GND #PWR709
+L GND #PWR0175
 U 1 1 54E94125
 P 8100 3800
-F 0 "#PWR709" H 8100 3550 60  0001 C CNN
+F 0 "#PWR0175" H 8100 3550 60  0001 C CNN
 F 1 "GND" H 8100 3650 60  0000 C CNN
 F 2 "" H 8100 3800 60  0000 C CNN

Commit message: placement completele! let the routing begin!
Connections:
- net labels added: RM, RXM, TM, TXM
Changed lines of the file:
@@
 Text Notes 5800 1900 0    60   ~ 0
 DIFF PAIR
+Text Label 2300 9000 1    60   ~ 0
+TXM
+Text Label 1900 9100 0    60   ~ 0
+RXM
+Text Label 2600 6700 0    60   ~ 0
+TM
+Text Label 2600 4700 0    60   ~ 0
+RM
 $EndSCHEMATC

Commit message: routed 98% of the CP, USB, ETH. normalized silk.
Connections:
- net labels added: EPHY_RES, ETH_SHELL
Changed lines of the file:
@@
 Text Label 2600 4700 0    60   ~ 0
 RM
+Text Label 5200 2700 0    60   ~ 0
+EPHY_RES
+Text Label 5200 8400 0    60   ~ 0
+ETH_SHELL
 $EndSCHEMATC
