File: tessel-v2-mediatek-usb.sch (KiCad schematic (older format))
At the start: 32 parts, among them J901 USB_A_2_stack, U201 MT7620N, U901 AIC1528-0PSTR, U902 FE1.1, X901 12MHz

Commit message: fully routed with sca/scl pulls
Parts:
- J901: footprint tm-kicad-lib:USB-double-xx-UAF-28 -> tm-kicad-lib:Molex-0672983090
Changed lines of the file:
@@
 $EndComp
 $Comp
-L GND #PWR0182
+L GND #PWR914
 U 1 1 54EDB81E
 P 9700 2800
-F 0 "#PWR0182" H 9700 2550 60  0001 C CNN
+F 0 "#PWR914" H 9700 2550 60  0001 C CNN
 F 1 "GND" H 9700 2650 60  0000 C CNN
 F 2 "" H 9700 2800 60  0000 C CNN
@@
 USB_18
 $Comp
-L GND #PWR0183
+L GND #PWR928
 U 1 1 54EDB969
 P 14300 4200
-F 0 "#PWR0183" H 14300 3950 60  0001 C CNN
+F 0 "#PWR928" H 14300 3950 60  0001 C CNN
 F 1 "GND" H 14300 4050 60  0000 C CNN
 F 2 "" H 14300 4200 60  0000 C CNN
@@
 $EndComp
 $Comp
-L GND #PWR0184
+L GND #PWR930
 U 1 1 54EDB9BA
 P 14700 4200
-F 0 "#PWR0184" H 14700 3950 60  0001 C CNN
+F 0 "#PWR930" H 14700 3950 60  0001 C CNN
 F 1 "GND" H 14700 4050 60  0000 C CNN
 F 2 "" H 14700 4200 60  0000 C CNN
@@
 $EndComp
 $Comp
-L GND #PWR0185
+L GND #PWR917
 U 1 1 54EDBA1F
 P 10700 8000
-F 0 "#PWR0185" H 10700 7750 60  0001 C CNN
+F 0 "#PWR917" H 10700 7750 60  0001 C CNN
 F 1 "GND" H 10700 7850 60  0000 C CNN
 F 2 "" H 10700 8000 60  0000 C CNN
@@
 $EndComp
 $Comp
-L +5V #PWR0186
+L +5V #PWR926
 U 1 1 54EA7C7D
 P 13900 3400
-F 0 "#PWR0186" H 13900 3250 60  0001 C CNN
+F 0 "#PWR926" H 13900 3250 60  0001 C CNN
 F 1 "+5V" H 13900 3540 60  0000 C CNN
 F 2 "" H 13900 3400 60  0000 C CNN
@@
 $EndComp
 $Comp
-L +5V #PWR0187
+L +5V #PWR902
 U 1 1 54EAE4B2
 P 1900 1500
-F 0 "#PWR0187" H 1900 1350 60  0001 C CNN
+F 0 "#PWR902" H 1900 1350 60  0001 C CNN
 F 1 "+5V" H 1900 1640 60  0000 C CNN
 F 2 "" H 1900 1500 60  0000 C CNN
@@
 VBUS[1]_IN
 $Comp
-L GND #PWR0188
+L GND #PWR909
 U 1 1 54EAE4FB
 P 6200 2700
-F 0 "#PWR0188" H 6200 2450 60  0001 C CNN
+F 0 "#PWR909" H 6200 2450 60  0001 C CNN
 F 1 "GND" H 6200 2550 60  0000 C CNN
 F 2 "" H 6200 2700 60  0000 C CNN
@@
 $EndComp
 $Comp
-L GND #PWR0189
+L GND #PWR912
 U 1 1 54EAE502
 P 7000 2700
-F 0 "#PWR0189" H 7000 2450 60  0001 C CNN
+F 0 "#PWR912" H 7000 2450 60  0001 C CNN
 F 1 "GND" H 7000 2550 60  0000 C CNN
 F 2 "" H 7000 2700 60  0000 C CNN
@@
 $EndComp
 $Comp
-L GND #PWR0190
+L GND #PWR908
 U 1 1 54EAE523
 P 6200 1600
-F 0 "#PWR0190" H 6200 1350 60  0001 C CNN
+F 0 "#PWR908" H 6200 1350 60  0001 C CNN
 F 1 "GND" H 6200 1450 60  0000 C CNN
 F 2 "" H 6200 1600 60  0000 C CNN
@@
 $EndComp
 $Comp
-L GND #PWR0191
+L GND #PWR911
 U 1 1 54EAE52A
 P 7000 1600
-F 0 "#PWR0191" H 7000 1350 60  0001 C CNN
+F 0 "#PWR911" H 7000 1350 60  0001 C CNN
 F 1 "GND" H 7000 1450 60  0000 C CNN
 F 2 "" H 7000 1600 60  0000 C CNN
@@
 $EndComp
 $Comp
-L GND #PWR0192
+L GND #PWR905
 U 1 1 54EAE531
 P 3500 2400
-F 0 "#PWR0192" H 3500 2150 60  0001 C CNN
+F 0 "#PWR905" H 3500 2150 60  0001 C CNN
 F 1 "GND" H 3500 2250 60  0000 C CNN
 F 2 "" H 3500 2400 60  0000 C CNN
@@
 NoConn ~ 11600 6300
 $Comp
-L GND #PWR0193
+L GND #PWR919
 U 1 1 54EB6EE4
 P 11100 4200
-F 0 "#PWR0193" H 11100 3950 60  0001 C CNN
+F 0 "#PWR919" H 11100 3950 60  0001 C CNN
 F 1 "GND" H 11100 4050 60  0000 C CNN
 F 2 "" H 11100 4200 60  0000 C CNN
@@
 $EndComp
 $Comp
-L GND #PWR0194
+L GND #PWR920
 U 1 1 54EB6F1C
 P 11500 4200
-F 0 "#PWR0194" H 11500 3950 60  0001 C CNN
+F 0 "#PWR920" H 11500 3950 60  0001 C CNN
 F 1 "GND" H 11500 4050 60  0000 C CNN
 F 2 "" H 11500 4200 60  0000 C CNN
@@
 $EndComp
 $Comp
-L GND #PWR0195
+L GND #PWR922
 U 1 1 54EB6F22
 P 11900 4200
-F 0 "#PWR0195" H 11900 3950 60  0001 C CNN
+F 0 "#PWR922" H 11900 3950 60  0001 C CNN
 F 1 "GND" H 11900 4050 60  0000 C CNN
 F 2 "" H 11900 4200 60  0000 C CNN
@@
 $EndComp
 $Comp
-L GND #PWR0196
+L GND #PWR923
 U 1 1 54EB6F5A
 P 12300 4200
-F 0 "#PWR0196" H 12300 3950 60  0001 C CNN
+F 0 "#PWR923" H 12300 3950 60  0001 C CNN
 F 1 "GND" H 12300 4050 60  0000 C CNN
 F 2 "" H 12300 4200 60  0000 C CNN
@@
 $EndComp
 $Comp
-L GND #PWR0197
+L GND #PWR925
 U 1 1 54EB8B85
 P 13900 2700
-F 0 "#PWR0197" H 13900 2450 60  0001 C CNN
+F 0 "#PWR925" H 13900 2450 60  0001 C CNN
 F 1 "GND" H 13900 2550 60  0000 C CNN
 F 2 "" H 13900 2700 60  0000 C CNN
@@
 $EndComp
 $Comp
-L GND #PWR0198
+L GND #PWR927
 U 1 1 54EB8B8B
 P 14300 2700
-F 0 "#PWR0198" H 14300 2450 60  0001 C CNN
+F 0 "#PWR927" H 14300 2450 60  0001 C CNN
 F 1 "GND" H 14300 2550 60  0000 C CNN
 F 2 "" H 14300 2700 60  0000 C CNN
@@
 $EndComp
 $Comp
-L GND #PWR0199
+L GND #PWR929
 U 1 1 54EB8B93
 P 14700 2700
-F 0 "#PWR0199" H 14700 2450 60  0001 C CNN
+F 0 "#PWR929" H 14700 2450 60  0001 C CNN
 F 1 "GND" H 14700 2550 60  0000 C CNN
 F 2 "" H 14700 2700 60  0000 C CNN
@@
 NoConn ~ 14600 7500
 $Comp
-L GND #PWR0200
+L GND #PWR921
 U 1 1 54EBFDB4
 P 11500 7600
-F 0 "#PWR0200" H 11500 7350 60  0001 C CNN
+F 0 "#PWR921" H 11500 7350 60  0001 C CNN
 F 1 "GND" H 11500 7450 60  0000 C CNN
 F 2 "" H 11500 7600 60  0000 C CNN
@@
 $EndComp
 $Comp
-L GND #PWR0201
+L GND #PWR918
 U 1 1 54EC0D43
 P 10700 10000
-F 0 "#PWR0201" H 10700 9750 60  0001 C CNN
+F 0 "#PWR918" H 10700 9750 60  0001 C CNN
 F 1 "GND" H 10700 9850 60  0000 C CNN
 F 2 "" H 10700 10000 60  0000 C CNN
@@
 $EndComp
 $Comp
-L GND #PWR0202
+L GND #PWR915
 U 1 1 54EC0DD4
 P 9700 10000
-F 0 "#PWR0202" H 9700 9750 60  0001 C CNN
+F 0 "#PWR915" H 9700 9750 60  0001 C CNN
 F 1 "GND" H 9700 9850 60  0000 C CNN
 F 2 "" H 9700 10000 60  0000 C CNN
@@
 $EndComp
 $Comp
-L GND #PWR0203
+L GND #PWR901
 U 1 1 54ECA394
 P 1700 5200
-F 0 "#PWR0203" H 1700 4950 60  0001 C CNN
+F 0 "#PWR901" H 1700 4950 60  0001 C CNN
 F 1 "GND" H 1700 5050 60  0000 C CNN
 F 2 "" H 1700 5200 60  0000 C CNN
@@
 $EndComp
 $Comp
-L +5V #PWR0204
+L +5V #PWR903
 U 1 1 54ECA39C
 P 2600 4800
-F 0 "#PWR0204" H 2600 4650 60  0001 C CNN
+F 0 "#PWR903" H 2600 4650 60  0001 C CNN
 F 1 "+5V" H 2600 4940 60  0000 C CNN
 F 2 "" H 2600 4800 60  0000 C CNN
@@
 $EndComp
 $Comp
-L GND #PWR0205
+L GND #PWR904
 U 1 1 54ECA3A8
 P 3000 5200
-F 0 "#PWR0205" H 3000 4950 60  0001 C CNN
+F 0 "#PWR904" H 3000 4950 60  0001 C CNN
 F 1 "GND" H 3000 5050 60  0000 C CNN
 F 2 "" H 3000 5200 60  0000 C CNN
@@
 $EndComp
 $Comp
-L +5V #PWR0206
+L +5V #PWR906
 U 1 1 54ECA3B0
 P 3900 4800
-F 0 "#PWR0206" H 3900 4650 60  0001 C CNN
+F 0 "#PWR906" H 3900 4650 60  0001 C CNN
 F 1 "+5V" H 3900 4940 60  0000 C CNN
 F 2 "" H 3900 4800 60  0000 C CNN
@@
 F 0 "J901" H 4350 4450 60  0000 C CNN
 F 1 "USB_A_2_stack" H 4950 3900 60  0000 C CNN
-F 2 "tm-kicad-lib:USB-double-xx-UAF-28" H 5800 4400 60  0001 C CNN
+F 2 "tm-kicad-lib:Molex-0672983090" H 5800 4400 60  0001 C CNN
 F 3 "" H 5800 4400 60  0000 C CNN
 	1    5000 3900
@@
 $EndComp
 $Comp
-L GND #PWR0207
+L GND #PWR907
 U 1 1 54ECA3BC
 P 5000 4800
-F 0 "#PWR0207" H 5000 4550 60  0001 C CNN
+F 0 "#PWR907" H 5000 4550 60  0001 C CNN
 F 1 "GND" H 5000 4650 60  0000 C CNN
 F 2 "" H 5000 4800 60  0000 C CNN
@@
 $EndComp
 $Comp
-L GND #PWR0208
+L GND #PWR910
 U 1 1 54ECA3C2
 P 6700 4500
-F 0 "#PWR0208" H 6700 4250 60  0001 C CNN
+F 0 "#PWR910" H 6700 4250 60  0001 C CNN
 F 1 "GND" H 6700 4350 60  0000 C CNN
 F 2 "" H 6700 4500 60  0000 C CNN
@@
 $EndComp
 $Comp
-L GND #PWR0209
+L GND #PWR924
 U 1 1 54ECF685
 P 12700 8100
-F 0 "#PWR0209" H 12700 7850 60  0001 C CNN
+F 0 "#PWR924" H 12700 7850 60  0001 C CNN
 F 1 "GND" H 12700 7950 60  0000 C CNN
 F 2 "" H 12700 8100 60  0000 C CNN
@@
 Connection ~ 13400 4600
 $Comp
-L +3.3V #PWR0210
+L +3.3V #PWR913
 U 1 1 54EDB88B
 P 8700 5000
-F 0 "#PWR0210" H 8700 4960 30  0001 C CNN
+F 0 "#PWR913" H 8700 4960 30  0001 C CNN
 F 1 "+3.3V" H 8700 5110 30  0000 C CNN
 F 2 "" H 8700 5000 60  0000 C CNN
@@
 	10400 5100 10400 5200
 $Comp
-L GND #PWR0211
+L GND #PWR916
 U 1 1 54ED096C
 P 10400 5200
-F 0 "#PWR0211" H 10400 4950 60  0001 C CNN
+F 0 "#PWR916" H 10400 4950 60  0001 C CNN
 F 1 "GND" H 10400 5050 60  0000 C CNN
 F 2 "" H 10400 5200 60  0000 C CNN
@@
 $EndComp
 $Comp
-L GND #PWR0212
+L GND #PWR931
 U 1 1 54ED10AE
 P 15100 2700
-F 0 "#PWR0212" H 15100 2450 60  0001 C CNN
+F 0 "#PWR931" H 15100 2450 60  0001 C CNN
 F 1 "GND" H 15100 2550 60  0000 C CNN
 F 2 "" H 15100 2700 60  0000 C CNN
