File: tessel-v2-mediatek-ram.sch (KiCad schematic (older format))
At the start: 21 parts, among them U201 MT7620N, U501 W9751G6KB-25

Commit message: swapped out all RLCs
Parts:
- C501, C502, C503, C504, C505, C506, C507, C508, C509, C510, C511, C512, C513, C514: symbol C -> TM_C
- R501, R502, R503, R504, R505: symbol R -> TM_R
Connections:
- wire segments 164 -> 221

Commit message: project save
Connections:
- wire segments 221 -> 164
Changed lines of the file:
@@
 DQS0
 $Comp
-L GND #PWR508
+L GND #PWR0131
 U 1 1 548D31D5
 P 13200 7200
-F 0 "#PWR508" H 13200 6950 60  0001 C CNN
+F 0 "#PWR0131" H 13200 6950 60  0001 C CNN
 F 1 "GND" H 13200 7050 60  0000 C CNN
 F 2 "" H 13200 7200 60  0000 C CNN
@@
 $EndComp
 $Comp
-L GND #PWR505
+L GND #PWR0132
 U 1 1 548D4FEE
 P 7900 3300
-F 0 "#PWR505" H 7900 3050 60  0001 C CNN
+F 0 "#PWR0132" H 7900 3050 60  0001 C CNN
 F 1 "GND" H 7900 3150 60  0000 C CNN
 F 2 "" H 7900 3300 60  0000 C CNN
@@
 $EndComp
 $Comp
-L +1.8V #PWR507
+L +1.8V #PWR0133
 U 1 1 5490BE7F
 P 11400 3000
-F 0 "#PWR507" H 11400 3140 20  0001 C CNN
+F 0 "#PWR0133" H 11400 3140 20  0001 C CNN
 F 1 "+1.8V" H 11400 3110 30  0000 C CNN
 F 2 "" H 11400 3000 60  0000 C CNN
@@
 $EndComp
 $Comp
-L +1.8V #PWR501
+L +1.8V #PWR0134
 U 1 1 5490C3F5
 P 2500 8400
-F 0 "#PWR501" H 2500 8540 20  0001 C CNN
+F 0 "#PWR0134" H 2500 8540 20  0001 C CNN
 F 1 "+1.8V" H 2500 8510 30  0000 C CNN
 F 2 "" H 2500 8400 60  0000 C CNN
@@
 $EndComp
 $Comp
-L +1.8V #PWR503
+L +1.8V #PWR0135
 U 1 1 5490C6A2
 P 7300 5300
-F 0 "#PWR503" H 7300 5440 20  0001 C CNN
+F 0 "#PWR0135" H 7300 5440 20  0001 C CNN
 F 1 "+1.8V" H 7300 5410 30  0000 C CNN
 F 2 "" H 7300 5300 60  0000 C CNN
@@
 $EndComp
 $Comp
-L GND #PWR504
+L GND #PWR0136
 U 1 1 54E9B31B
 P 7700 7300
-F 0 "#PWR504" H 7700 7050 60  0001 C CNN
+F 0 "#PWR0136" H 7700 7050 60  0001 C CNN
 F 1 "GND" H 7700 7150 60  0000 C CNN
 F 2 "" H 7700 7300 60  0000 C CNN
@@
 DDR_VREF
 $Comp
-L GND #PWR502
+L GND #PWR0137
 U 1 1 54EB9E52
 P 6100 9400
-F 0 "#PWR502" H 6100 9150 60  0001 C CNN
+F 0 "#PWR0137" H 6100 9150 60  0001 C CNN
 F 1 "GND" H 6100 9250 60  0000 C CNN
 F 2 "" H 6100 9400 60  0000 C CNN
@@
 CKE
 $Comp
-L GND #PWR506
+L GND #PWR0138
 U 1 1 54E8D57D
 P 7900 4500
-F 0 "#PWR506" H 7900 4250 60  0001 C CNN
+F 0 "#PWR0138" H 7900 4250 60  0001 C CNN
 F 1 "GND" H 7900 4350 60  0000 C CNN
 F 2 "" H 7900 4500 60  0000 C CNN
@@
 	11500 7000 11500 7100
 Wire Wire Line
-	11500 7100 11600 7100
-Wire Wire Line
-	11600 7100 11700 7100
-Wire Wire Line
-	11700 7100 11800 7100
-Wire Wire Line
-	11800 7100 11900 7100
-Wire Wire Line
-	11900 7100 12100 7100
-Wire Wire Line
-	12100 7100 12200 7100
-Wire Wire Line
-	12200 7100 12300 7100
-Wire Wire Line
-	12300 7100 12400 7100
-Wire Wire Line
-	12400 7100 12500 7100
-Wire Wire Line
-	12500 7100 12600 7100
-Wire Wire Line
-	12600 7100 12700 7100
-Wire Wire Line
-	12700 7100 12800 7100
-Wire Wire Line
-	12800 7100 12900 7100
-Wire Wire Line
-	12900 7100 13000 7100
-Wire Wire Line
-	13000 7100 13200 7100
+	11500 7100 13200 7100
 Wire Wire Line
 	11600 7100 11600 7000
@@
 Connection ~ 12200 7100
 Wire Wire Line
-	13200 7000 13200 7100
-Wire Wire Line
-	13200 7100 13200 7200
+	13200 7000 13200 7200
 Wire Wire Line
 	12400 7100 12400 7000
@@
 	4500 5600 5400 5600
 Wire Wire Line
-	7700 2500 7900 2500
-Wire Wire Line
-	7900 2500 8400 2500
-Wire Wire Line
-	8400 2500 9200 2500
+	7700 2500 9200 2500
 Wire Wire Line
 	7900 2600 7900 2500
@@
 	6200 3700 7100 3700
 Wire Wire Line
-	11400 3100 11500 3100
-Wire Wire Line
-	11500 3100 11600 3100
-Wire Wire Line
-	11600 3100 11700 3100
-Wire Wire Line
-	11700 3100 11800 3100
-Wire Wire Line
-	11800 3100 12000 3100
-Wire Wire Line
-	12000 3100 12100 3100
-Wire Wire Line
-	12100 3100 12200 3100
-Wire Wire Line
-	12200 3100 12300 3100
-Wire Wire Line
-	12300 3100 12400 3100
-Wire Wire Line
-	12400 3100 12500 3100
-Wire Wire Line
-	12500 3100 12600 3100
-Wire Wire Line
-	12600 3100 12700 3100
-Wire Wire Line
-	12700 3100 12800 3100
-Wire Wire Line
-	12800 3100 12900 3100
-Wire Wire Line
-	12900 3100 13100 3100
-Wire Wire Line
-	11400 3000 11400 3100
-Wire Wire Line
-	11400 3100 11400 3200
+	11400 3100 13100 3100
+Wire Wire Line
+	11400 3000 11400 3200
 Wire Wire Line
 	11500 3200 11500 3100
@@
 Connection ~ 12900 3100
 Wire Wire Line
-	2500 8400 2500 8500
-Wire Wire Line
-	2500 8500 2500 8600
-Wire Wire Line
-	2500 8500 2900 8500
-Wire Wire Line
-	2900 8500 3300 8500
-Wire Wire Line
-	3300 8500 3700 8500
-Wire Wire Line
-	3700 8500 4100 8500
-Wire Wire Line
-	4100 8500 4500 8500
-Wire Wire Line
-	4500 8500 4900 8500
-Wire Wire Line
-	4900 8500 5300 8500
-Wire Wire Line
-	5300 8500 5700 8500
-Wire Wire Line
-	5700 8500 6100 8500
+	2500 8400 2500 8600
+Wire Wire Line
+	2500 8500 6100 8500
 Wire Wire Line
 	2900 8500 2900 8600
@@
 	4100 9300 4100 9200
 Wire Wire Line
-	2500 9300 2900 9300
-Wire Wire Line
-	2900 9300 3300 9300
-Wire Wire Line
-	3300 9300 3700 9300
-Wire Wire Line
-	3700 9300 4100 9300
-Wire Wire Line
-	4100 9300 4500 9300
-Wire Wire Line
-	4500 9300 4900 9300
-Wire Wire Line
-	4900 9300 5300 9300
-Wire Wire Line
-	5300 9300 5700 9300
-Wire Wire Line
-	5700 9300 6100 9300
+	2500 9300 6100 9300
 Wire Wire Line
 	3700 9300 3700 9200
@@
 Connection ~ 5700 8500
 Wire Wire Line
-	6100 9200 6100 9300
-Wire Wire Line
-	6100 9300 6100 9400
+	6100 9200 6100 9400
 Wire Wire Line
 	5700 9300 5700 9200
@@
 Connection ~ 4900 9300
 Wire Wire Line
-	7300 5300 7300 5400
-Wire Wire Line
-	7300 5400 7300 5500
+	7300 5300 7300 5500
 Wire Wire Line
 	7700 5400 7700 5500
 Wire Wire Line
-	7700 6100 7700 6300
-Wire Wire Line
-	7700 6300 7700 6400
-Wire Wire Line
-	7700 6400 7700 6500
-Wire Wire Line
-	7300 6100 7300 6400
-Wire Wire Line
-	7300 6400 7300 6500
+	7700 6100 7700 6500
+Wire Wire Line
+	7300 6100 7300 6500
 Wire Wire Line
 	7300 6400 7700 6400
@@
 Connection ~ 13200 7100
 Wire Wire Line
-	7700 7100 7700 7200
-Wire Wire Line
-	7700 7200 7700 7300
+	7700 7100 7700 7300
 Wire Wire Line
 	7300 7200 7700 7200
@@
 	10900 4400 10100 4400
 Wire Wire Line
-	7700 3700 7900 3700
-Wire Wire Line
-	7900 3700 8400 3700
-Wire Wire Line
-	8400 3700 9200 3700
+	7700 3700 9200 3700
 Wire Wire Line
 	7900 3700 7900 3800
